File: hardware/HEF Sensor.kicad_sch (KiCad schematic)
At the start: 7 parts, among them J9 Conn_01x03_Socket, U23 WCS1700, U24 ADR02AUJZ

Commit message: Fixed massive GitHub confusion.
Parts:
- renumbered C23 to C14, C24 to C15, C25 to C16, J9 to J6, TP4 to TP1, U23 to U17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
